Commit message: URDF now resembles the real robot

File: ros/src/laser_description/urdf/laser.xacro (robot description, xacro)
@@ -13,9 +13,10 @@
             <origin rpy="0 0 0" xyz="0 0 -0.0015"/>
             <geometry>
-                <box size="${base_link_length} ${base_link_width} 0.003"/>
+                <box size="${metal_plate_length} ${metal_plate_width} 0.003"/>
             </geometry>
             <material name="blue"/>
         </visual>
     </link>
+    <!-- Rotary Table -->
     <link name="rotary_base">
         <visual>
@@ -29,9 +30,9 @@
     <joint name="base_link__rotary_base" type="fixed">
         <axis xyz="0 0 1" />
-        <origin rpy="0 0 0" xyz="0 0 0"/>
+        <origin rpy="0 0 0" xyz="0.020 0 0"/>
         <parent link="base_link"/>
         <child link="rotary_base"/>
     </joint>
-    <link name="rotary_invisible">
+    <link name="rotary_base_invisible">
         <visual>
             <origin rpy="0 0 0" xyz="0 0 0"/>
@@ -41,8 +42,8 @@
         </visual>
     </link>
-    <joint name="rotary_base__rotary_invisible" type="fixed">
+    <joint name="rotary_base__rotary_base_invisible" type="fixed">
         <origin rpy="1.57 0 0" xyz="0 0 0"/>
         <parent link="rotary_base"/>
-        <child link="rotary_invisible"/>
+        <child link="rotary_base_invisible"/>
     </joint>
     <link name="rotary_middle">
@@ -55,12 +56,13 @@
         </visual>
     </link>
-    <joint name="rotary_base__rotary_middle" type="revolute">
+    <joint name="A" type="revolute">
         <axis xyz="1 0 0" />
-        <limit effort="1000.0" lower="-2.356" upper="0" velocity="0.5" />
-        <origin rpy="0 0 0" xyz="0 0.08 0"/>
-        <parent link="rotary_invisible"/>
+        <limit effort="1000.0" lower="${theta4_limit}" upper="0" velocity="1" />
+        <origin rpy="0 0 0" xyz="0 ${metal_plate_to_rotary_center_height} 0"/>
+        <parent link="rotary_base_invisible"/>
         <child link="rotary_middle"/>
     </joint>
-    <link name="rotary_top">
+    <!-- rotary_top = Work Coordinate Frame -->
+    <link name="W">
         <visual>
             <origin rpy="0 0 0" xyz="0 0 0"/>
@@ -71,18 +73,12 @@
         </visual>
     </link>
-    <joint name="rotary_middle__rotary_top" type="revolute">
+    <joint name="B" type="revolute">
         <axis xyz="0 0 1" />
-        <limit effort="1000.0" lower="-314" upper="0" velocity="0.5" />
-        <origin rpy="0 0 0" xyz="0 0 0.120"/>
+        <limit effort="1000.0" lower="${theta5_limit}" upper="0" velocity="1" />
+        <origin rpy="0 0 0" xyz="0 0 ${rotary_center_to_rotary_top}"/>
         <parent link="rotary_middle"/>
-        <child link="rotary_top"/>
+        <child link="W"/>
     </joint>
-    <!-- <joint name="base_link__tool" type="revolute">
-        <axis xyz="0 0 1" />
-        <limit effort="1000.0" lower="-3.14" upper="3.14" velocity="0.5" />
-        <origin rpy="0 0 0" xyz="2.0 1.2 0.5"/>
-        <parent link="base_link"/>
-        <child link="tool"/>
-    </joint> -->
+    <!-- Linear Stage -->
     <link name="y_box1">
         <visual>
@@ -93,9 +89,9 @@
         </visual>
     </link>
-    <joint name="base_link__y_box1" type="prismatic">
+    <joint name="Z" type="prismatic">
         <axis xyz="0 0 1" />
-        <limit effort="1000.0" lower="${-z_joint_limit}" upper="0" velocity="0.5" />
-        <origin rpy="0 0 0" xyz="${x_rail_length/2+rail_width} ${base_link_width-y_rail_length} 0.3"/>
-        <parent link="base_link"/>
+        <limit effort="1000.0" lower="${d3_limit}" upper="0" velocity="1" />
+        <origin rpy="0 0 0" xyz="${rotary_center_to_linear_stage_x} ${rotary_center_to_linear_stage_y} ${metal_plate_to_rotary_center_height+rotary_center_to_linear_stage_z}"/>
+        <parent link="rotary_base"/>
         <child link="y_box1"/>
     </joint>
@@ -121,12 +117,13 @@
         </visual>
     </link>
-    <joint name="y_box1__x_box" type="prismatic">
+    <joint name="Y" type="prismatic">
         <axis xyz="0 1 0" />
-        <limit effort="1000.0" lower="-0.26" upper="0" velocity="0.5" />
+        <limit effort="1000.0" lower="${d2_limit}" upper="0" velocity="1" />
         <origin rpy="0 0 3.1415" xyz="${-rail_width/2} 0.09 ${rail_width}"/>
         <parent link="y_box1"/>
         <child link="x_box"/>
     </joint>
-    <link name="tool">
+    <!-- tool = Tool Coordinates Frame -->
+    <link name="T">
         <visual>
             <origin rpy="0 0 0" xyz="0 0 ${laser_height/2}"/>
@@ -137,10 +134,10 @@
         </visual>
     </link>
-    <joint name="x_box__tool" type="prismatic">
+    <joint name="X" type="prismatic">
         <axis xyz="1 0 0" />
-        <limit effort="1000.0" lower="-0.26" upper="0" velocity="0.5" />
+        <limit effort="1000.0" lower="${d1_limit}" upper="0" velocity="1" />
         <origin rpy="0 0 3.1415" xyz="0.063 ${rail_width/2+laser_rad} ${rail_width/2-laser_height}"/>
         <parent link="x_box"/>
-        <child link="tool"/>
+        <child link="T"/>
     </joint>
 </robot>

File: ros/src/laser_description/urdf/robot_parameters.xacro (robot description, xacro)
@@ -1,6 +1,12 @@
 <?xml version="1.0" ?>
 <robot xmlns:xacro="http://www.ros.org/wiki/xacro">
-  <xacro:property name="base_link_length" value="0.43"/>
-  <xacro:property name="base_link_width" value="0.20"/>
+  <!-- Modele Parameters -->
+  <xacro:property name="metal_plate_length" value="0.43"/>
+  <xacro:property name="metal_plate_width" value="0.20"/>
+  <xacro:property name="metal_plate_to_rotary_center_height" value="0.080"/>
+  <xacro:property name="rotary_center_to_rotary_top" value="0.13145"/>
+  <xacro:property name="rotary_center_to_linear_stage_x" value="0.1845"/>
+  <xacro:property name="rotary_center_to_linear_stage_y" value="-0.2653"/>
+  <xacro:property name="rotary_center_to_linear_stage_z" value="0.2426"/>
   <xacro:property name="laser_rad" value="0.015"/>
   <xacro:property name="laser_height" value="0.069"/>
@@ -8,5 +14,12 @@
   <xacro:property name="rail_width" value="0.04"/>
   <xacro:property name="y_rail_length" value="0.42"/>
-  <xacro:property name="z_joint_limit" value="0.069"/>
   <xacro:property name="x_rail_length" value="0.347"/>
+  <!-- Joint Parameters -->
+  <xacro:property name="d1_limit" value="-0.280"/>
+  <xacro:property name="d2_limit" value="-0.280"/>
+  <xacro:property name="d3_limit" value="-0.065"/>
+  <!-- theta4 joint limit = 150 deg -->
+  <xacro:property name="theta4_limit" value="-2.617"/>
+  <!-- theta5 joint no limit -->
+  <xacro:property name="theta5_limit" value="-62.8"/>
 </robot>

Commit message: calibrate robot

File: ros/src/laser_description/urdf/laser.xacro (robot description, xacro)
@@ -58,5 +58,5 @@
     <joint name="A" type="revolute">
         <axis xyz="1 0 0" />
-        <limit effort="1000.0" lower="${theta4_limit}" upper="0" velocity="1" />
+        <limit effort="1000.0" lower="${A_limit}" upper="0" velocity="1" />
         <origin rpy="0 0 0" xyz="0 ${metal_plate_to_rotary_center_height} 0"/>
         <parent link="rotary_base_invisible"/>
@@ -75,5 +75,5 @@
     <joint name="B" type="revolute">
         <axis xyz="0 0 1" />
-        <limit effort="1000.0" lower="${theta5_limit}" upper="0" velocity="1" />
+        <limit effort="1000.0" lower="${B_limit}" upper="0" velocity="1" />
         <origin rpy="0 0 0" xyz="0 0 ${rotary_center_to_rotary_top}"/>
         <parent link="rotary_middle"/>
@@ -91,6 +91,6 @@
     <joint name="Z" type="prismatic">
         <axis xyz="0 0 1" />
-        <limit effort="1000.0" lower="${d3_limit}" upper="0" velocity="1" />
-        <origin rpy="0 0 0" xyz="${rotary_center_to_linear_stage_x} ${rotary_center_to_linear_stage_y} ${metal_plate_to_rotary_center_height+rotary_center_to_linear_stage_z}"/>
+        <limit effort="1000.0" lower="${Z_limit}" upper="0" velocity="1" />
+        <origin rpy="0 0 0" xyz="${rotary_center_to_linear_stage_x + X_joint_offset + rail_width/2} ${rotary_center_to_linear_stage_y - Y_joint_offset + rail_width/2 + laser_rad} ${metal_plate_to_rotary_center_height + rotary_center_to_linear_stage_z + laser_height - 1.5*rail_width}"/>
         <parent link="rotary_base"/>
         <child link="y_box1"/>
@@ -119,6 +119,6 @@
     <joint name="Y" type="prismatic">
         <axis xyz="0 1 0" />
-        <limit effort="1000.0" lower="${d2_limit}" upper="0" velocity="1" />
-        <origin rpy="0 0 3.1415" xyz="${-rail_width/2} 0.09 ${rail_width}"/>
+        <limit effort="1000.0" lower="${Y_limit}" upper="0" velocity="1" />
+        <origin rpy="0 0 3.1415" xyz="${-rail_width/2} ${Y_joint_offset} ${rail_width}"/>
         <parent link="y_box1"/>
         <child link="x_box"/>
@@ -136,6 +136,6 @@
     <joint name="X" type="prismatic">
         <axis xyz="1 0 0" />
-        <limit effort="1000.0" lower="${d1_limit}" upper="0" velocity="1" />
-        <origin rpy="0 0 3.1415" xyz="0.063 ${rail_width/2+laser_rad} ${rail_width/2-laser_height}"/>
+        <limit effort="1000.0" lower="${X_limit}" upper="0" velocity="1" />
+        <origin rpy="0 0 3.1415" xyz="${X_joint_offset} ${rail_width/2+laser_rad} ${rail_width/2-laser_height}"/>
         <parent link="x_box"/>
         <child link="T"/>

File: ros/src/laser_description/urdf/robot_parameters.xacro (robot description, xacro)
@@ -1,25 +1,24 @@
 <?xml version="1.0" ?>
 <robot xmlns:xacro="http://www.ros.org/wiki/xacro">
-  <!-- Modele Parameters -->
+  <!-- Modele Parameters (m)-->
   <xacro:property name="metal_plate_length" value="0.43"/>
   <xacro:property name="metal_plate_width" value="0.20"/>
   <xacro:property name="metal_plate_to_rotary_center_height" value="0.080"/>
-  <xacro:property name="rotary_center_to_rotary_top" value="0.11045"/>
-  <xacro:property name="rotary_center_to_linear_stage_x" value="0.1845"/>
-  <xacro:property name="rotary_center_to_linear_stage_y" value="-0.2653"/>
-  <xacro:property name="rotary_center_to_linear_stage_z" value="0.2426"/>
+  <xacro:property name="rotary_center_to_rotary_top" value="0.1263"/>
+  <xacro:property name="rotary_center_to_linear_stage_x" value="0.102"/>
+  <xacro:property name="rotary_center_to_linear_stage_y" value="-0.207"/>
+  <xacro:property name="rotary_center_to_linear_stage_z" value="0.2186"/>
   <xacro:property name="laser_rad" value="0.015"/>
   <xacro:property name="laser_height" value="0.069"/>
-  <xacro:property name="laser_pos_from_plate" value="0.3"/>
   <xacro:property name="rail_width" value="0.04"/>
   <xacro:property name="y_rail_length" value="0.42"/>
   <xacro:property name="x_rail_length" value="0.347"/>
   <!-- Joint Parameters -->
-  <xacro:property name="d1_limit" value="-0.280"/>
-  <xacro:property name="d2_limit" value="-0.280"/>
-  <xacro:property name="d3_limit" value="-0.065"/>
-  <!-- theta4 joint limit = 150 deg -->
-  <xacro:property name="theta4_limit" value="-2.617"/>
-  <!-- theta5 joint no limit -->
-  <xacro:property name="theta5_limit" value="-62.8"/>
+  <xacro:property name="X_limit" value="-0.290"/>
+  <xacro:property name="Y_limit" value="-0.280"/>
+  <xacro:property name="Z_limit" value="-0.065"/>
+  <xacro:property name="A_limit" value="-2.617"/>
+  <xacro:property name="B_limit" value="-62.8"/>
+  <xacro:property name="Y_joint_offset" value="0.08"/>
+  <xacro:property name="X_joint_offset" value="0.03"/>
 </robot>
